Commit message: Fix: Integrate SICK lidar driver as standard folder, tune Nav2, and update launch files

File: src/amr_mp_description/description/lidar.xacro (robot description, xacro)
@@ -3,8 +3,8 @@
     <joint name="laser_joint" type="fixed">
         <parent link="chassis"/>
-        <child  link="laser_frame"/>
-        <origin xyz="0.25 0 0.175" rpy="0 0 -1.5708"/>
+        <child  link="laser_link"/>
+        <origin xyz="0.25 0 0.175" rpy="0 0 0"/>
     </joint>
-    <link name="laser_frame">
+    <link name="laser_link">
         <visual>
             <geometry><cylinder radius="0.05" length="0.04"/></geometry>
